Commit message: positioning done: 1.2 Ohter Objects in kitchen

File: cob_gazebo_objects/objects/expedit_white_ikea_shelf.urdf (robot description, URDF)
Before this commit: robot Bett_Fjellse, 1 links, 0 joints
Links:
- link base_link: geometry collision box size=0.41 0.79 1.49; visual mesh filename=package://cob_gazebo_objects/Media/models/expedit_white_ike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
