Commit message: positioning done: Kitchen Table and Chairs, Partition Walls, Objects on Kitchen Table. Modified: IPA ikea table now with textures, apple_juice_box now with cap, partiton wall 8 added.

File: cob_gazebo_objects/objects/apple_juice_box.urdf (robot description, URDF)
Before this commit: robot my_object, 1 links, 0 joints
Links:
- link base_link: mass 1.036 -> 0.475; geometry collision box size=0.062 0.07 0.251; visual mesh filename=package://cob_gazebo_objects/Media/models/apple_juice_box.d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

File: cob_gazebo_objects/objects/table_ikea.urdf.xacro (robot description, xacro)
@@ -29,10 +29,10 @@
                izz="0" />
     </inertial>
-    <visual>
+<visual>
       <origin xyz="0.0 0.0 ${table_z+table_height-table_top_thickness/2}" />
       <geometry>
         <box size="${table_width} ${table_depth} ${table_top_thickness}" />
       </geometry>
-    </visual>
+</visual>
     <collision>
       <origin xyz="0.0 0.0 ${table_z+table_height-table_top_thickness/2}" />
@@ -43,5 +43,5 @@
   </link>
   <gazebo reference="table_top_link">
-    <material>Gazebo/White</material>
+    <material>kitchen_white</material>
     <mu1>50.0</mu1>
     <mu2>50.0</mu2>
@@ -71,6 +71,6 @@
             </collision>
         </link>
-	<gazebo reference="legs">
-		<material>Gazebo/White</material>
+	<gazebo reference="leg_${suffix}_link">
+		<material>kitchen_white</material>
 		<turnGravityOff>false</turnGravityOff>
 	</gazebo>
@@ -107,6 +107,6 @@
             </collision>
         </link>
-	<gazebo reference="structure_lath">
-		<material>Gazebo/White</material>
+	<gazebo reference="lath_${suffix}_link">
+		<material>kitchen_white</material>
 		<turnGravityOff>false</turnGravityOff>
 	</gazebo>
