Commit message: positioning done: all objects in livingroom. spawn files updated. new objects added.

File: cob_gazebo_objects/objects/beer_hofbraeu.urdf (robot description, URDF)
Before this commit: robot my_object, 1 links, 0 joints
Links:
- link base_link: mass 1.0 -> 0.370; geometry collision box size=0.065 0.065 0.26; visual mesh filename=package://cob_gazebo_objects/Media/models/beer_hofbraeu.dae

File: cob_gazebo_objects/objects/beer_rothaus.urdf (robot description, URDF)
Before this commit: robot my_object, 1 links, 0 joints
Links:
- link base_link: mass 1.0 -> 0.370; geometry collision box size=0.055 0.055 0.23; visual mesh filename=package://cob_gazebo_objects/Media/models/beer_rothaus.dae

File: cob_gazebo_objects/objects/blue_white_tray.urdf (robot description, URDF)
Before this commit: robot my_object, 1 links, 0 joints
Links:
- link base_link: mass 1.0 -> 0.400; geometry collision box size=0.37 0.50 0.02; visual mesh filename=package://cob_gazebo_objects/Media/models/blue_white_tray.d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

File: cob_gazebo_objects/objects/couch.urdf.xacro (robot description, xacro)
@@ -189,3 +189,6 @@
 		<child link="right_couch_middle" />
 	</joint>
+<gazebo>
+	<static>true</static>
+</gazebo>
 </robot>

File: cob_gazebo_objects/objects/green_tea3.urdf (robot description, URDF)
Before this commit: robot my_object, 1 links, 0 joints
Links:
- link base_link: mass 1.0 -> 1.37; geometry collision box size=0.057 0.091 0.195; visual mesh filename=package://cob_gazebo_objects/Media/models/green_tea.dae

File: cob_gazebo_objects/objects/large_carton_empty.urdf (robot description, URDF)
Before this commit: robot my_object, 1 links, 0 joints
Links:
- link base_link: mass 1.0 -> 0.500; geometry collision mesh filename=package://cob_gazebo_objects/Media/models/large_carton_empt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; visual mesh filename=package://cob_gazebo_objects/Media/models/large_carton_empt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

File: cob_gazebo_objects/objects/pizza_box.urdf (robot description, URDF)
Before this commit: robot my_object, 1 links, 0 joints
Links:
- link base_link: mass 1.0 -> 0.700; geometry collision box size=0.41 0.60 0.035; visual mesh filename=package://cob_gazebo_objects/Media/models/pizza_box.dae

File: cob_gazebo_objects/objects/pizza_box2.urdf (robot description, URDF)
Before this commit: robot my_object, 1 links, 0 joints
Links:
- link base_link: mass 1.0 -> 0.700; geometry collision box size=0.41 0.60 0.035; visual mesh filename=package://cob_gazebo_objects/Media/models/pizza_box.dae

File: cob_gazebo_objects/objects/sliding_door.urdf (robot description, URDF)
Before this commit: robot my_object, 1 links, 0 joints
Links:
- link base_link: geometry collision mesh filename=package://cob_gazebo_objects/Media/models/sliding_door.dae; visual mesh filename=package://cob_gazebo_objects/Media/models/sliding_door.dae

File: cob_gazebo_objects/objects/styroprene.urdf (robot description, URDF)
Before this commit: robot my_object, 1 links, 0 joints
Links:
- link base_link: mass 1.0 -> 0.200; geometry collision box size=0.30 0.30 0.08; visual mesh filename=package://cob_gazebo_objects/Media/models/styroprene.dae
