Commit message: positioning done: all objects in bedroom. spawn files updated. new objects added.

File: cob_gazebo_objects/objects/Bett_Fjellse_middlePillow.urdf (robot description, URDF)
Before this commit: robot Bett_Fjellse, 1 links, 0 joints
Links:
- link base_link: mass 1.0 -> 20.0; geometry collision mesh filename=package://cob_gazebo_objects/Media/models/Bett_Fjellse_boun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; visual mesh filename=package://cob_gazebo_objects/Media/models/Bett_Fjellse_midd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

File: cob_gazebo_objects/objects/corn_flakes_package2.urdf (robot description, URDF)
Before this commit: robot Bett_Fjellse, 1 links, 0 joints
Links:
- link base_link: mass 1.0 -> 0.445; geometry collision box size=0.068 0.192 0.29; visual mesh filename=package://cob_gazebo_objects/Media/models/corn_flakes_packa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

File: cob_gazebo_objects/objects/pringles_red.urdf (robot description, URDF)
Before this commit: robot Bett_Fjellse, 1 links, 0 joints
Links:
- link base_link: mass 1.0 -> 0.045; geometry collision box size=0.075 0.075 0.23; visual mesh filename=package://cob_gazebo_objects/Media/models/pringles_red.dae
