Commit message: bugs fixed: fixed positioning of some objects, fixed spawn files, added new SRS_divider6

File: cob_gazebo_objects/objects/SRS_divider8.urdf (robot description, URDF)
Before this commit: robot my_object, 1 links, 0 joints
Links:
- link base_link: geometry collision mesh filename=package://cob_gazebo_objects/Media/models/SRS_divider6.dae; visual mesh filename=package://cob_gazebo_objects/Media/models/SRS_divider6.dae
