Commit message: big plants now have correct (round) boundings for laser scanner detection. possible through automatic bounding box + modified bounding collada

File: cob_gazebo_objects/objects/large_plant_big.urdf (robot description, URDF)
Before this commit: robot my_object, 1 links, 0 joints
Links:
- link base_link: geometry collision mesh filename=package://cob_gazebo_objects/Media/models/large_plant_big_b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; visual mesh filename=package://cob_gazebo_objects/Media/models/large_plant_big.d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

File: cob_gazebo_objects/objects/large_plant_small.urdf (robot description, URDF)
Before this commit: robot my_object, 1 links, 0 joints
Links:
- link base_link: geometry collision mesh filename=package://cob_gazebo_objects/Media/models/large_plant_small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; visual mesh filename=package://cob_gazebo_objects/Media/models/large_plant_small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
