Commit message: dust mop bounding box, two objects static, deleted old launchfiles/locationfiles

File: cob_gazebo_objects/objects/dust_mop.urdf (robot description, URDF)
Before this commit: robot my_object, 1 links, 0 joints
Links:
- link base_link: geometry collision box size=0.095 1.50 0.052; visual mesh filename=package://cob_gazebo_objects/Media/models/dust_mop.dae

Commit message: adjusted bounding box of dust_mop using custom joints

File: cob_gazebo_objects/objects/dust_mop.urdf (robot description, URDF)
Before this commit: robot my_object, 1 links, 0 joints
Links:
- added link base_addition, mass 0; collision box size=0.05 0.001 0.010; visual box size=0 0 0
- added link base_addition2, mass 0; collision box size=0.103 0.0013 0.010; visual box size=0 0 0
- added link stick, mass 0; collision cylinder length=1.355 radius=0.013; visual cylinder length=1.355 radius=0.013
- link base_link: geometry collision box size=0.095 0.38 0.01; visual mesh filename=package://cob_gazebo_objects/Media/models/dust_mop.dae
Joints:
- added joint base_to_base_addition: type fixed, parent base_link, child base_addition
- added joint base_to_base_addition2: type fixed, parent base_link, child base_addition2
- added joint base_to_stick: type fixed, parent base_link, child stick

Commit message: model modified: dust_mop

File: cob_gazebo_objects/objects/dust_mop.urdf (robot description, URDF)
Before this commit: robot my_object, 4 links, 3 joints
Links:
- link stick: geometry collision cylinder length=1.355 radius=0.013; visual cylinder length=0 radius=0
