Commit message: corrected door_bedroom appearence

File: cob_gazebo_objects/objects/door_white_bedroom.urdf (robot description, URDF)
Before this commit: robot my_object, 1 links, 0 joints
Links:
- link base_link: geometry collision mesh filename=package://cob_gazebo_objects/Media/models/door_white_bedroo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; visual mesh filename=package://cob_gazebo_objects/Media/models/door_white_bedroo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
