Commit message: screw updated in terms of actual model

File: cob_gazebo_objects/objects/screw.urdf (robot description, URDF)
Before this commit: robot screw, 2 links, 1 joints
Links:
- link body: geometry collision cylinder length=0.035 radius=0.004; visual cylinder length=0.035 radius=0.004
- link head: geometry collision cylinder length=0.0025 radius=0.01; visual cylinder length=0.0025 radius=0.01

Commit message: Scenario Update, two screw_boxes on table, one of them filled with screws

File: cob_gazebo_objects/objects/screw.urdf (robot description, URDF)
Before this commit: robot screw, 2 links, 1 joints
Links:
- link body: mass .0125 -> .0005
- link head: mass .0125 -> .0005

File: cob_gazebo_objects/objects/simple_screwbox.urdf (robot description, URDF)
Before this commit: robot simple_screwbox, 7 links, 10 joints
Links:
- link base: mass 1.0 -> 5.0
- link retainer_ew: mass .0125 -> .125
- link retainer_hc: mass .0125 -> .125
- link retainer_nw: mass .0125 -> .125
- link retainer_sw: mass .0125 -> .125
- link retainer_vc: mass .0125 -> .125
- link retainer_ww: mass .0125 -> .125

File: cob_gazebo_objects/objects/table_ikea.urdf.xacro (robot description, xacro)
@@ -23,9 +23,9 @@
   <link name="table_top_link">
     <inertial>
-      <mass value="5.0" />
+      <mass value="10.0" />
       <origin xyz="0.0 0.0 0.0" />
-      <inertia ixx="0" ixy="0"  ixz="0"
-               iyy="0" iyz="0"
-               izz="0" />
+      <inertia ixx="100.0" ixy="0"  ixz="0"
+               iyy="100.0" iyz="0"
+               izz="100.0" />
     </inertial>
     <visual>
@@ -43,5 +43,5 @@
   </link>
   <gazebo reference="table_top_link">
-    <material>Gazebo/White</material>
+    <material>IPA/Cabinet_Wood</material>
     <mu1>50.0</mu1>
     <mu2>50.0</mu2>
@@ -54,7 +54,7 @@
 		<origin xyz="0 0 0" />
                 <mass value="3" />
-                <inertia  ixx="0" ixy="0" ixz="0"
-                          iyy="0" iyz="0"
-                          izz="0" />
+                <inertia  ixx="100.0" ixy="0" ixz="0"
+                          iyy="100.0" iyz="0"
+                          izz="100.0" />
             </inertial>
             <visual>
@@ -72,5 +72,5 @@
         </link>
 	<gazebo reference="legs">
-		<material>Gazebo/White</material>
+		<material>IPA/Cabinet_Wood</material>
 		<turnGravityOff>false</turnGravityOff>
 	</gazebo>
@@ -90,7 +90,7 @@
 		<origin xyz="0 0 0" />
                 <mass value="1" />
-                <inertia  ixx="0" ixy="0" ixz="0"
-                          iyy="0" iyz="0"
-                          izz="0" />
+                <inertia  ixx="10.0" ixy="0" ixz="0"
+                          iyy="10.0" iyz="0"
+                          izz="10.0" />
             </inertial>
             <visual>
@@ -108,5 +108,5 @@
         </link>
 	<gazebo reference="structure_lath">
-		<material>Gazebo/White</material>
+		<material>IPA/Cabinet_Wood</material>
 		<turnGravityOff>false</turnGravityOff>
 	</gazebo>
