Commit message: Second (working) version for new objects in PRACE

File: cob_gazebo_objects/objects/simple_screwbox.urdf (robot description, URDF)
Before this commit: robot simple_screwbox, 7 links, 10 joints
Links:
- link base: geometry collision box size=.10 .10 .050; visual box size=.10 .10 .050
- link retainer_ew: geometry collision box size=0.005 0.04 0.02; visual box size=0.005 0.04 0.02
- link retainer_hc: geometry collision box size=0.04 0.01 0.02; visual box size=0.04 0.01 0.02
- link retainer_nw: geometry collision box size=0.05 0.005 0.02; visual box size=0.05 0.005 0.02
- link retainer_sw: geometry collision box size=0.05 0.005 0.02; visual box size=0.05 0.005 0.02
- link retainer_vc: geometry collision box size=0.01 0.04 0.02; visual box size=0.01 0.04 0.02
- link retainer_ww: geometry collision box size=0.005 0.04 0.02; visual box size=0.005 0.04 0.02

Commit message: simple_screwbox updated in terms of actual model

File: cob_gazebo_objects/objects/simple_screwbox.urdf (robot description, URDF)
Before this commit: robot simple_screwbox, 7 links, 10 joints
Links:
- link retainer_ew: geometry collision box size=0.0055 0.035 0.02; visual box size=0.0055 0.035 0.02
- link retainer_hc: geometry collision box size=0.035 0.015 0.02; visual box size=0.035 0.015 0.02
- link retainer_nw: geometry collision box size=0.045 0.0055 0.02; visual box size=0.045 0.0055 0.02
- link retainer_sw: geometry collision box size=0.045 0.0055 0.02; visual box size=0.045 0.0055 0.02
- link retainer_vc: geometry collision box size=0.015 0.035 0.02; visual box size=0.015 0.035 0.02
- link retainer_ww: geometry collision box size=0.0055 0.035 0.02; visual box size=0.0055 0.035 0.02

Commit message: updated scenario

File: cob_gazebo_objects/objects/simple_screwbox.urdf (robot description, URDF)
Before this commit: robot simple_screwbox, 7 links, 10 joints
Links:
- link base: geometry collision box size=.075 .075 .010; visual box size=.075 .075 .010
