Commit message: 3D map updated, basmati rice textures fixed.

File: cob_gazebo_worlds/urdf/ipa-apartment/landing.urdf.xacro (robot description, xacro)
@@ -83,5 +83,5 @@
 	</gazebo>
 	<joint name="joint_wall_ext2" type="fixed">
-		<origin xyz="8.70 -2.565 ${size_z_wall1/2}" rpy="0 0 0" />
+		<origin xyz="8.70 -1.565 ${size_z_wall1/2}" rpy="0 0 0" />
 		<parent link="origin_landing" />
 		<child link="wall_ext2" />
@@ -298,12 +298,12 @@
 			<origin xyz="0 0 0" />
 			<geometry>
-				<box size="1.73 ${wall_depth} ${size_z_wall1}" />
-			</geometry>
-			<material name="IPA/Grey"/>
-		</visual>
-		<collision>
-			<origin xyz="0 0 0" />
-			<geometry>
-				<box size="1.73 ${wall_depth} ${size_z_wall1}" />
+				<box size="1.96 ${wall_depth} ${size_z_wall1}" />
+			</geometry>
+			<material name="IPA/Grey"/>
+		</visual>
+		<collision>
+			<origin xyz="0 0 0" />
+			<geometry>
+				<box size="1.96 ${wall_depth} ${size_z_wall1}" />
 			</geometry>
 		</collision>
@@ -313,5 +313,5 @@
 	</gazebo>
 	<joint name="joint_wall_ext10" type="fixed">
-		<origin xyz="2.005 7.53 ${size_z_wall1/2}" rpy="0 0 0" />
+		<origin xyz="1.89 7.53 ${size_z_wall1/2}" rpy="0 0 0" />
 		<parent link="origin_landing" />
 		<child link="wall_ext10" />
@@ -369,5 +369,5 @@
 	</gazebo>
 	<joint name="joint_wall_ext12" type="fixed">
-		<origin xyz="1.18 6.908 ${size_z_wall1/2}" rpy="0 0 0" />
+		<origin xyz="0.95 6.908 ${size_z_wall1/2}" rpy="0 0 0" />
 		<parent link="origin_landing" />
 		<child link="wall_ext12" />
