Commit message: fixes for spawn-scripts and worlds (unrecognized textures)

File: cob_gazebo_worlds/urdf/ipa-apartment/apartment.urdf.xacro (robot description, xacro)
@@ -17,5 +17,5 @@
 				<box size="${wall_depth} ${size_d+0.18+0.35} ${size_z_wall1}" />
 			</geometry>
-			<material name="Grey"/>
+			<material name="IPA/Grey"/>
 		</visual>
 		<collision>
@@ -46,5 +46,5 @@
 				<box size=" ${size_b} 0.001 0.90" />
 			</geometry>
-			<material name="Grey"/>
+			<material name="IPA/Grey"/>
 		</visual>
 		<collision>
@@ -75,5 +75,5 @@
 				<box size=" ${size_b} 0.35 0.90" />
 			</geometry>
-			<material name="Grey"/>
+			<material name="IPA/Grey"/>
 		</visual>
 		<collision>
@@ -104,5 +104,5 @@
 				<box size="0.02 0.35 2.70" />
 			</geometry>
-			<material name="Grey"/>
+			<material name="IPA/Grey"/>
 		</visual>
 		<collision>
@@ -133,5 +133,5 @@
 				<box size=" ${size_b} ${window_depth} 1.80" />
 			</geometry>
-			<material name="Grey"/>
+			<material name="IPA/Grey"/>
 		</visual>
 		<collision>
@@ -162,5 +162,5 @@
 				<box size="${wall_depth} ${size_a+0.35} ${size_z_wall2}" />
 			</geometry>
-			<material name="Grey"/>
+			<material name="IPA/Grey"/>
 		</visual>
 		<collision>
@@ -191,5 +191,5 @@
 				<box size=" ${window_depth} 1.4 ${size_z_wall2}" />
 			</geometry>
-			<material name="Grey"/>
+			<material name="IPA/Grey"/>
 		</visual>
 		<collision>
@@ -220,5 +220,5 @@
 				<box size="${window_depth} 1.6 ${size_z_wall2}" />
 			</geometry>
-			<material name="Grey"/>
+			<material name="IPA/Grey"/>
 		</visual>
 		<collision>
@@ -249,5 +249,5 @@
 				<box size="${wall_depth} ${size_a} ${size_z_wall2}" />
 			</geometry>
-			<material name="Grey"/>
+			<material name="IPA/Grey"/>
 		</visual>
 		<collision>
@@ -278,5 +278,5 @@
 				<box size=" ${size_b} ${window_depth} ${size_z_wall2}" />
 			</geometry>
-			<material name="Grey"/>
+			<material name="IPA/Grey"/>
 		</visual>
 		<collision>
@@ -308,5 +308,5 @@
 				<box size="${wall_depth} ${size_a} ${size_z_wall1}" />
 			</geometry>
-			<material name="Grey"/>
+			<material name="IPA/Grey"/>
 		</visual>
 		<collision>
@@ -337,5 +337,5 @@
 				<box size="${wall_depth} 1.9 ${size_z_wall2}" />
 			</geometry>
-			<material name="Grey"/>
+			<material name="IPA/Grey"/>
 		</visual>
 		<collision>
@@ -367,5 +367,5 @@
 				<box size=" ${size_b-0.1} 0.02 ${size_z_wall2}" />
 			</geometry>
-			<material name="Grey"/>
+			<material name="IPA/Grey"/>
 		</visual>
 		<collision>
@@ -384,6 +384,6 @@
 		<child link="wall_09" />
 	</joint>
-	<!-- glas_00 -->
-	<link name="glas_00">
+	<!-- glass_00 -->
+	<link name="glass_00">
 		<inertial>
 			<origin xyz="0 0 0" />
@@ -396,5 +396,5 @@
 				<box size="0.02 0.62 ${size_z_wall1}" />
 			</geometry>
-			<material name="Transparent"/>
+			<material name="IPA/Grey"/>
 		</visual>
 		<collision>
@@ -405,14 +405,14 @@
 		</collision>
 	</link>
-	<gazebo reference="glas_00">
+	<gazebo reference="glass_00">
 		<material>IPA/Wall2</material>
 	</gazebo>
-	<joint name="joint_glas_00" type="fixed">
+	<joint name="joint_glass_00" type="fixed">
 		<origin xyz="${-size_total_x/2+dist_axis_x-wall_depth} ${1.23-dist_axis_y-0.09} ${size_z_wall1/2}" rpy="0 0 0" />
 		<parent link="dummy_link" />
-		<child link="glas_00" />
-	</joint>
-<!-- glas_00_aluminium_part -->
-	<link name="glas_00_aluminium_part">
+		<child link="glass_00" />
+	</joint>
+<!-- glass_00_aluminium_part -->
+	<link name="glass_00_aluminium_part">
 		<inertial>
 			<origin xyz="0 0 0" />
@@ -425,5 +425,5 @@
 				<box size="0.03 0.62 0.10" />
 			</geometry>
-			<material name="Transparent"/>
+			<material name="IPA/Grey"/>
 		</visual>
 		<collision>
@@ -434,14 +434,14 @@
 		</collision>
 	</link>
-	<gazebo reference="glas_00_aluminium_part">
+	<gazebo reference="glass_00_aluminium_part">
 		<material>aluminium</material>
 	</gazebo>
-	<joint name="joint_glas_00_aluminium_part" type="fixed">
+	<joint name="joint_glass_00_aluminium_part" type="fixed">
 		<origin xyz="${-size_total_x/2+dist_axis_x-wall_depth} ${1.23-dist_axis_y-0.09} 0.05" rpy="0 0 0" />
 		<parent link="dummy_link" />
-		<child link="glas_00_aluminium_part" />
-	</joint>
-	<!-- glas_01 -->
-	<link name="glas_01">
+		<child link="glass_00_aluminium_part" />
+	</joint>
+	<!-- glass_01 -->
+	<link name="glass_01">
 		<inertial>
 			<origin xyz="0 0 0" />
@@ -454,5 +454,5 @@
 				<box size="0.02 0.92 ${size_z_wall1}" />
 			</geometry>
-			<material name="Transparent"/>
+			<material name="IPA/Grey"/>
 		</visual>
 		<collision>
@@ -463,14 +463,14 @@
 		</collision>
 	</link>
-	<gazebo reference="glas_01">
+	<gazebo reference="glass_01">
 		<material>IPA/Wall2</material>
 	</gazebo>
-	<joint name="joint_glas_01" type="fixed">
+	<joint name="joint_glass_01" type="fixed">
 		<origin xyz="${-size_total_x/2+dist_axis_x-wall_depth} ${-0.68-dist_axis_y} ${size_z_wall1/2}" rpy="0 0 0" />
 		<parent link="dummy_link" />
-		<child link="glas_01" />
-	</joint>
-<!-- glas_01_aluminium_part -->
-	<link name="glas_01_aluminium_part">
+		<child link="glass_01" />
+	</joint>
+<!-- glass_01_aluminium_part -->
+	<link name="glass_01_aluminium_part">
 		<inertial>
 			<origin xyz="0 0 0" />
@@ -483,5 +483,5 @@
 				<box size="0.03 0.92 0.10" />
 			</geometry>
-			<material name="Transparent"/>
+			<material name="IPA/Grey"/>
 		</visual>
 		<collision>
@@ -492,14 +492,14 @@
 		</collision>
 	</link>
-	<gazebo reference="glas_01_aluminium_part">
+	<gazebo reference="glass_01_aluminium_part">
 		<material>aluminium</material>
 	</gazebo>
-	<joint name="joint_glas_01_aluminium_part" type="fixed">
+	<joint name="joint_glass_01_aluminium_part" type="fixed">
 		<origin xyz="${-size_total_x/2+dist_axis_x-wall_depth} ${-0.68-dist_axis_y} 0.05" rpy="0 0 0" />
 		<parent link="dummy_link" />
-		<child link="glas_01_aluminium_part" />
-	</joint>
-	<!-- glasdoor -->
-	<link name="glasdoor">
+		<child link="glass_01_aluminium_part" />
+	</joint>
+	<!-- glassdoor -->
+	<link name="glassdoor">
 		<inertial>
 			<origin xyz="0 0 0" />
@@ -512,5 +512,5 @@
 				<box size="1.00 0.02 ${size_z_wall1}" />
 			</geometry>
-			<material name="Transparent"/>
+			<material name="IPA/Grey"/>
 		</visual>
 		<collision>
@@ -521,14 +521,14 @@
 		</collision>
 	</link>
-	<gazebo reference="glasdoor">
+	<gazebo reference="glassdoor">
 		<material>IPA/Wall2</material>
 	</gazebo>
-	<joint name="glasdoor" type="fixed">
+	<joint name="glassdoor" type="fixed">
 		<origin xyz="-2.63 -4.27 ${size_z_wall1/2}" rpy="0 0 0" />
 		<parent link="dummy_link" />
-		<child link="glasdoor" />
-	</joint>
-	<!-- glasdoor_aluminum_part -->
-	<link name="glasdoor_aluminum_part">
+		<child link="glassdoor" />
+	</joint>
+	<!-- glassdoor_aluminum_part -->
+	<link name="glassdoor_aluminum_part">
 		<inertial>
 			<origin xyz="0 0 0" />
@@ -541,5 +541,5 @@
 				<box size="1.00 0.03 0.10" />
 			</geometry>
-			<material name="Transparent"/>
+			<material name="IPA/Grey"/>
 		</visual>
 		<collision>
@@ -550,11 +550,11 @@
 		</collision>
 	</link>
-	<gazebo reference="glasdoor_aluminum_part">
+	<gazebo reference="glassdoor_aluminum_part">
 		<material>aluminium</material>
 	</gazebo>
-	<joint name="glasdoor_aluminum_part" type="fixed">
+	<joint name="glassdoor_aluminum_part" type="fixed">
 		<origin xyz="-2.63 -4.27 0.05" rpy="0 0 0" />
 		<parent link="dummy_link" />
-		<child link="glasdoor_aluminum_part" />
+		<child link="glassdoor_aluminum_part" />
 	</joint>
         </xacro:macro>

File: cob_gazebo_worlds/urdf/ipa-apartment/elevator.urdf.xacro (robot description, xacro)
@@ -80,5 +80,5 @@
 				<box size="2.4 0.04 ${size_z_wall1}" />
 			</geometry>
-			<material name="Grey"/>
+			<material name="IPA/Grey"/>
 		</visual>
 		<collision>
@@ -109,5 +109,5 @@
 				<box size="2.4 0.04 ${size_z_wall1}" />
 			</geometry>
-			<material name="Grey"/>
+			<material name="IPA/Grey"/>
 		</visual>
 		<collision>
@@ -138,5 +138,5 @@
 				<box size="0.04 0.87 ${size_z_wall1}" />
 			</geometry>
-			<material name="Grey"/>
+			<material name="IPA/Grey"/>
 		</visual>
 		<collision>
@@ -206,5 +206,5 @@
 				<box size="2.4 0.04 ${size_z_wall1}" />
 			</geometry>
-			<material name="Grey"/>
+			<material name="IPA/Grey"/>
 		</visual>
 		<collision>
@@ -235,5 +235,5 @@
 				<box size="2.4 0.04 ${size_z_wall1}" />
 			</geometry>
-			<material name="Grey"/>
+			<material name="IPA/Grey"/>
 		</visual>
 		<collision>
@@ -264,5 +264,5 @@
 				<box size="0.04 0.87 ${size_z_wall1}" />
 			</geometry>
-			<material name="Grey"/>
+			<material name="IPA/Grey"/>
 		</visual>
 		<collision>
@@ -382,5 +382,5 @@
 				<box size="0.04 1.74 ${size_z_wall1}" />
 			</geometry>
-			<material name="Grey"/>
+			<material name="IPA/Grey"/>
 		</visual>
 		<collision>
@@ -410,5 +410,5 @@
 				<box size="0.04 1.74 ${size_z_wall1}" />
 			</geometry>
-			<material name="Grey"/>
+			<material name="IPA/Grey"/>
 		</visual>
 		<collision>
@@ -438,5 +438,5 @@
 				<box size="0.04 1.3 ${size_z_wall1}" />
 			</geometry>
-			<material name="Grey"/>
+			<material name="IPA/Grey"/>
 		</visual>
 		<collision>

File: cob_gazebo_worlds/urdf/ipa-apartment/landing.urdf.xacro (robot description, xacro)
@@ -41,5 +41,5 @@
 				<box size="2.1 ${wall_depth} ${size_z_wall1}" />
 			</geometry>
-			<material name="Grey"/>
+			<material name="IPA/Grey"/>
 		</visual>
 		<collision>
@@ -70,5 +70,5 @@
 				<box size="2.2 ${wall_depth} ${size_z_wall1}" />
 			</geometry>
-			<material name="Grey"/>
+			<material name="IPA/Grey"/>
 		</visual>
 		<collision>
@@ -99,5 +99,5 @@
 				<box size="${wall_depth} 1.73 ${size_z_wall1}" />
 			</geometry>
-			<material name="Grey"/>
+			<material name="IPA/Grey"/>
 		</visual>
 		<collision>
@@ -128,5 +128,5 @@
 				<box size="${wall_depth} 1.73 ${size_z_wall1}" />
 			</geometry>
-			<material name="Grey"/>
+			<material name="IPA/Grey"/>
 		</visual>
 		<collision>
@@ -156,5 +156,5 @@
 				<box size="1.25 ${wall_depth} ${size_z_wall1}" />
 			</geometry>
-			<material name="Grey"/>
+			<material name="IPA/Grey"/>
 		</visual>
 		<collision>
@@ -184,5 +184,5 @@
 				<box size="1.25 ${wall_depth} ${size_z_wall1}" />
 			</geometry>
-			<material name="Grey"/>
+			<material name="IPA/Grey"/>
 		</visual>
 		<collision>
@@ -213,5 +213,5 @@
 				<box size="${wall_depth} 2.1 ${size_z_wall1}" />
 			</geometry>
-			<material name="Grey"/>
+			<material name="IPA/Grey"/>
 		</visual>
 		<collision>
@@ -242,5 +242,5 @@
 				<box size="${wall_depth} 2.3 ${size_z_wall1}" />
 			</geometry>
-			<material name="Grey"/>
+			<material name="IPA/Grey"/>
 		</visual>
 		<collision>
@@ -271,5 +271,5 @@
 				<box size="1.73 ${wall_depth} ${size_z_wall1}" />
 			</geometry>
-			<material name="Grey"/>
+			<material name="IPA/Grey"/>
 		</visual>
 		<collision>
@@ -300,5 +300,5 @@
 				<box size="1.73 ${wall_depth} ${size_z_wall1}" />
 			</geometry>
-			<material name="Grey"/>
+			<material name="IPA/Grey"/>
 		</visual>
 		<collision>
@@ -328,5 +328,5 @@
 				<box size="${wall_depth} 1.30 ${size_z_wall1}" />
 			</geometry>
-			<material name="Grey"/>
+			<material name="IPA/Grey"/>
 		</visual>
 		<collision>
@@ -356,5 +356,5 @@
 				<box size="${wall_depth} 1.30 ${size_z_wall1}" />
 			</geometry>
-			<material name="Grey"/>
+			<material name="IPA/Grey"/>
 		</visual>
 		<collision>
@@ -385,5 +385,5 @@
 				<box size="${wall_depth} 6.6 ${size_z_wall1}" />
 			</geometry>
-			<material name="Grey"/>
+			<material name="IPA/Grey"/>
 		</visual>
 		<collision>
@@ -415,5 +415,5 @@
 				<box size="${wall_depth} 6.6 ${size_z_wall1}" />
 			</geometry>
-			<material name="Grey"/>
+			<material name="IPA/Grey"/>
 		</visual>
 		<collision>
@@ -445,5 +445,5 @@
 				<box size="${wall_depth} 6.6 ${size_z_wall1}" />
 			</geometry>
-			<material name="Grey"/>
+			<material name="IPA/Grey"/>
 		</visual>
 		<collision>
@@ -475,5 +475,5 @@
 				<box size="${wall_depth} 1.8 ${size_z_wall1}" />
 			</geometry>
-			<material name="Grey"/>
+			<material name="IPA/Grey"/>
 		</visual>
 		<collision>
@@ -505,5 +505,5 @@
 				<box size="1.8 ${wall_depth} ${size_z_wall1}" />
 			</geometry>
-			<material name="Grey"/>
+			<material name="IPA/Grey"/>
 		</visual>
 		<collision>
@@ -534,5 +534,5 @@
 				<box size="${wall_depth} 6.75 ${size_z_wall1}" />
 			</geometry>
-			<material name="Grey"/>
+			<material name="IPA/Grey"/>
 		</visual>
 		<collision>
@@ -562,5 +562,5 @@
 				<box size="0.06 6.00 ${size_z_wall2}" />
 			</geometry>
-			<material name="Grey"/>
+			<material name="IPA/Grey"/>
 		</visual>
 		<collision>
@@ -590,5 +590,5 @@
 				<box size="1.2 ${wall_depth} ${size_z_wall1}" />
 			</geometry>
-			<material name="Grey"/>
+			<material name="IPA/Grey"/>
 		</visual>
 		<collision>
@@ -618,5 +618,5 @@
 				<box size="1.99 0.06 ${size_z_wall1}" />
 			</geometry>
-			<material name="Grey"/>
+			<material name="IPA/Grey"/>
 		</visual>
 		<collision>
@@ -647,5 +647,5 @@
 				<box size="${wall_depth} 1.1 ${size_z_wall1}" />
 			</geometry>
-			<material name="Grey"/>
+			<material name="IPA/Grey"/>
 		</visual>
 		<collision>
@@ -676,5 +676,5 @@
 				<box size="${wall_depth} 0.23 ${size_z_wall1}" />
 			</geometry>
-			<material name="Grey"/>
+			<material name="IPA/Grey"/>
 		</visual>
 		<collision>
@@ -705,5 +705,5 @@
 				<box size="0.35 0.35 ${size_z_wall1}" />
 			</geometry>
-			<material name="Grey"/>
+			<material name="IPA/Grey"/>
 		</visual>
 		<collision>

File: cob_gazebo_worlds/urdf/ipa-apartment/office.urdf.xacro (robot description, xacro)
@@ -41,5 +41,5 @@
 				<box size="2.8 ${wall_depth} ${size_z_wall1}" />
 			</geometry>
-			<material name="Grey"/>
+			<material name="IPA/Grey"/>
 		</visual>
 		<collision>
@@ -70,5 +70,5 @@
 				<box size="4.4 ${wall_depth} ${size_z_wall1}" />
 			</geometry>
-			<material name="Grey"/>
+			<material name="IPA/Grey"/>
 		</visual>
 		<collision>
@@ -99,5 +99,5 @@
 				<box size="0.26 5.3 ${size_z_wall2}" />
 			</geometry>
-			<material name="Grey"/>
+			<material name="IPA/Grey"/>
 		</visual>
 		<collision>
@@ -129,5 +129,5 @@
 				<box size="${wall_depth} 8.2 ${size_z_wall2}" />
 			</geometry>
-			<material name="Grey"/>
+			<material name="IPA/Grey"/>
 		</visual>
 		<collision>
@@ -159,5 +159,5 @@
 				<box size="2.2 ${wall_depth} ${size_z_wall2}" />
 			</geometry>
-			<material name="Grey"/>
+			<material name="IPA/Grey"/>
 		</visual>
 		<collision>
@@ -189,5 +189,5 @@
 				<box size="${wall_depth} 4.21 ${size_z_wall1}" />
 			</geometry>
-			<material name="Grey"/>
+			<material name="IPA/Grey"/>
 		</visual>
 		<collision>
@@ -218,5 +218,5 @@
 				<box size="${wall_depth} 1.40 ${size_z_wall1}" />
 			</geometry>
-			<material name="Grey"/>
+			<material name="IPA/Grey"/>
 		</visual>
 		<collision>
@@ -247,5 +247,5 @@
 				<box size="${wall_depth} 2.0 ${size_z_wall1}" />
 			</geometry>
-			<material name="Grey"/>
+			<material name="IPA/Grey"/>
 		</visual>
 		<collision>
@@ -276,5 +276,5 @@
 				<box size="${wall_depth} 0.3 ${size_z_wall1}" />
 			</geometry>
-			<material name="Grey"/>
+			<material name="IPA/Grey"/>
 		</visual>
 		<collision>
@@ -305,5 +305,5 @@
 				<box size="4.53 ${wall_depth} ${size_z_wall1}" />
 			</geometry>
-			<material name="Grey"/>
+			<material name="IPA/Grey"/>
 		</visual>
 		<collision>
@@ -334,5 +334,5 @@
 				<box size="4.5 ${wall_depth} ${size_z_wall1}" />
 			</geometry>
-			<material name="Grey"/>
+			<material name="IPA/Grey"/>
 		</visual>
 		<collision>
@@ -364,5 +364,5 @@
 				<box size="${wall_depth} 3.80 ${size_z_wall1}" />
 			</geometry>
-			<material name="Grey"/>
+			<material name="IPA/Grey"/>
 		</visual>
 		<collision>
@@ -393,5 +393,5 @@
 				<box size="${wall_depth} 0.52 ${size_z_wall1}" />
 			</geometry>
-			<material name="Grey"/>
+			<material name="IPA/Grey"/>
 		</visual>
 		<collision>
@@ -422,5 +422,5 @@
 				<box size="0.001 2.6 0.90" />
 			</geometry>
-			<material name="Grey"/>
+			<material name="IPA/Grey"/>
 		</visual>
 		<collision>
@@ -451,5 +451,5 @@
 				<box size="0.35 2.6 0.90" />
 			</geometry>
-			<material name="Grey"/>
+			<material name="IPA/Grey"/>
 		</visual>
 		<collision>
@@ -480,5 +480,5 @@
 				<box size="${window_depth} 2.6 1.80" />
 			</geometry>
-			<material name="Grey"/>
+			<material name="IPA/Grey"/>
 		</visual>
 		<collision>
@@ -497,5 +497,5 @@
 		<child link="wall_office_13_part3" />
 	</joint>
-<!-- wall_office_13_part4 (little glas)-->
+<!-- wall_office_13_part4 (little glass)-->
 	<link name="wall_office_13_part4">
 		<inertial>
@@ -509,5 +509,5 @@
 				<box size="0.35 0.02 1.80" />
 			</geometry>
-			<material name="Grey"/>
+			<material name="IPA/Grey"/>
 		</visual>
 		<collision>
@@ -538,5 +538,5 @@
 				<box size="1.9 ${wall_depth} ${size_z_wall2}" />
 			</geometry>
-			<material name="Grey"/>
+			<material name="IPA/Grey"/>
 		</visual>
 		<collision>
@@ -567,5 +567,5 @@
 				<box size="5.0 ${wall_depth} ${size_z_wall2}" />
 			</geometry>
-			<material name="Grey"/>
+			<material name="IPA/Grey"/>
 		</visual>
 		<collision>
@@ -596,5 +596,5 @@
 				<box size="1.6 ${wall_depth} ${size_z_wall1}" />
 			</geometry>
-			<material name="Grey"/>
+			<material name="IPA/Grey"/>
 		</visual>
 		<collision>
@@ -625,5 +625,5 @@
 				<box size="0.26 0.26 ${size_z_wall1}" />
 			</geometry>
-			<material name="Grey"/>
+			<material name="IPA/Grey"/>
 		</visual>
 		<collision>
@@ -654,5 +654,5 @@
 				<box size="${wall_depth} 1.15 ${size_z_wall1}" />
 			</geometry>
-			<material name="Grey"/>
+			<material name="IPA/Grey"/>
 		</visual>
 		<collision>
@@ -683,5 +683,5 @@
 				<box size="${wall_depth} 1.08 ${size_z_wall1}" />
 			</geometry>
-			<material name="Grey"/>
+			<material name="IPA/Grey"/>
 		</visual>
 		<collision>
@@ -712,5 +712,5 @@
 				<box size="${wall_depth} 1.10 ${size_z_wall1}" />
 			</geometry>
-			<material name="Grey"/>
+			<material name="IPA/Grey"/>
 		</visual>
 		<collision>

File: cob_gazebo_worlds/urdf/ipa-apartment/wall_ipa.urdf.xacro (robot description, xacro)
@@ -16,5 +16,5 @@
 				<box size="0.77 0.10 2.40" />
 			</geometry>
-			<material name="Grey"/>
+			<material name="IPA/Grey"/>
 		</visual>
 		<collision>

Commit message: :q

File: cob_gazebo_worlds/urdf/ipa-apartment/apartment.urdf.xacro (robot description, xacro)
@@ -32,5 +32,5 @@
   </joint>
   <!-- wall_01 -->
-  <link name="wall_01">
+  <link name="wall_01_part1">
     <inertial>
       <origin xyz="0 0 0" />
@@ -52,11 +52,11 @@
     </collision>
   </link>
-  <gazebo reference="wall_01">
+  <gazebo reference="wall_01_part1">
     <material>kitchen_wall_with_heating</material>
   </gazebo>
-  <joint name="joint_wall_01" type="fixed">
+  <joint name="joint_wall_01_part1" type="fixed">
     <origin xyz="${dist_axis_x} ${size_total_y/2-dist_axis_y+window_depth+0.02} 0.45" rpy="0 0 0" />
     <parent link="dummy_link" />
-    <child link="wall_01" />
+    <child link="wall_01_part1" />
   </joint>
   <!-- wall_01_part2 -->

File: cob_gazebo_worlds/urdf/ipa-apartment/landing.urdf.xacro (robot description, xacro)
@@ -56,5 +56,5 @@
   </joint-->
   <!-- wall ext -->
-  <link name="wall_ext2">
+  <link name="door_E334">
     <inertial>
       <origin xyz="0 0 0" />
@@ -76,11 +76,11 @@
     </collision>
   </link>
-  <gazebo reference="wall_ext2">
+  <gazebo reference="door_E334">
     <material>door_E334</material>
   </gazebo>
-  <joint name="joint_wall_ext2" type="fixed">
+  <joint name="joint_door_E334" type="fixed">
     <origin xyz="8.70 -1.565 ${size_z_wall1/2}" rpy="0 0 0" />
     <parent link="origin_landing" />
-    <child link="wall_ext2" />
+    <child link="door_E334" />
   </joint>
   <!-- wall ext -->
